File: SythesizerKiCAD/synthesizer.kicad_pcb (KiCad board)
At the start: 2 copper layers, 98.2 x 95.2 mm, 86 parts, among them U2 LM1877, U3 LMC6484

Commit message: Frequencies and timer periods
Parts:
- MSP430FR1: footprint Package_QFP:LQFP-48-1EP_7x7mm_P0.5mm_EP3.6x3.6mm -> Package_QFP:LQFP-48_7x7mm_P0.5mm
Changed lines of the file:
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@@
       (outputformat 1)
       (mirror false)
-      (drillshape 1)
+      (drillshape 0)
       (scaleselection 1)
-      (outputdirectory "")
+      (outputdirectory "../Gerbers/")
     )
   )
@@
     )
   )
-  (footprint "Package_QFP:LQFP-48-1EP_7x7mm_P0.5mm_EP3.6x3.6mm" (layer "F.Cu")
+  (footprint "Package_QFP:LQFP-48_7x7mm_P0.5mm" (layer "F.Cu")
     (at 76.24 90.25)
-    (descr "LQFP, 48 Pin (http://www.analog.com/media/en/technical-documentation/data-sheets/LTC7810.pdf), generated with kicad-footprint-generator ipc_gullwing_generator.py")
+    (descr "LQFP, 48 Pin (https://www.analog.com/media/en/technical-documentation/data-sheets/ltc2358-16.pdf), generated with kicad-footprint-generator ipc_gullwing_generator.py")
     (tags "LQFP QFP")
     (property "Sheetfile" "synthesizer.kicad_sch")
@@
         (effects (font (size 1 1) (thickness 0.15)))
     )
-    (fp_text value "~" (at 0 5.85) (layer "F.Fab") hide
+    (fp_text value "~" (at 0 5.85) (layer "F.Fab")
         (effects (font (size 1 1) (thickness 0.15)))
     )
@@
     (fp_line (start 3.5 3.5) (end -3.5 3.5)
       (stroke (width 0.1) (type solid)) (layer "F.Fab"))
-    (pad "" smd roundrect (at -1.2 -1.2) (size 0.97 0.97) (layers "F.Paste") (roundrect_rratio 0.25))
-    (pad "" smd roundrect (at -1.2 0) (size 0.97 0.97) (layers "F.Paste") (roundrect_rratio 0.25))
-    (pad "" smd roundrect (at -1.2 1.2) (size 0.97 0.97) (layers "F.Paste") (roundrect_rratio 0.25))
-    (pad "" smd roundrect (at 0 -1.2) (size 0.97 0.97) (layers "F.Paste") (roundrect_rratio 0.25))
-    (pad "" smd roundrect (at 0 0) (size 0.97 0.97) (layers "F.Paste") (roundrect_rratio 0.25))
-    (pad "" smd roundrect (at 0 1.2) (size 0.97 0.97) (layers "F.Paste") (roundrect_rratio 0.25))
-    (pad "" smd roundrect (at 1.2 -1.2) (size 0.97 0.97) (layers "F.Paste") (roundrect_rratio 0.25))
-    (pad "" smd roundrect (at 1.2 0) (size 0.97 0.97) (layers "F.Paste") (roundrect_rratio 0.25))
-    (pad "" smd roundrect (at 1.2 1.2) (size 0.97 0.97) (layers "F.Paste") (roundrect_rratio 0.25))
     (pad "1" smd roundrect (at -4.1625 -2.75) (size 1.475 0.3) (layers "F.Cu" "F.Paste" "F.Mask") (roundrect_rratio 0.25)
       (net 14 "/P1.2") (pinfunction "P1.2/UCB0SIMO/UCB0SDA/TB0TRG/OA0-/A2/Veref-") (pintype "bidirectional"))
@@
     (pad "48" smd roundrect (at -2.75 -4.1625) (size 0.3 1.475) (layers "F.Cu" "F.Paste" "F.Mask") (roundrect_rratio 0.25)
       (net 12 "/P1.3") (pinfunction "1.3/UCB0SOMI/UCB0SCL/A3") (pintype "bidirectional"))
-    (pad "49" smd rect (at 0 0) (size 3.6 3.6) (layers "F.Cu" "F.Mask"))
-    (model "${KICAD6_3DMODEL_DIR}/Package_QFP.3dshapes/LQFP-48-1EP_7x7mm_P0.5mm_EP3.6x3.6mm.wrl"
+    (model "${KICAD6_3DMODEL_DIR}/Package_QFP.3dshapes/LQFP-48_7x7mm_P0.5mm.wrl"
       (offset (xyz 0 0 0))
       (scale (xyz 1 1 1))
@@
     (fp_circle (center 0 0) (end 1.75 0)
       (stroke (width 0.1) (type solid)) (fill none) (layer "F.Fab"))
-    (pad "1" thru_hole roundrect (at 0 0) (size 3.5 3.5) (drill 1.55) (layers "*.Cu" "*.Mask") (roundrect_rratio 0.071429)
+    (pad "1" thru_hole roundrect (at 0 0) (size 3.5 3.5) (drill 1.55) (layers "*.Cu" "*.Mask") (roundrect_rratio 0.07142914286)
       (net 60 "/Audio_Out"))
     (model "${KICAD6_3DMODEL_DIR}/Connector_Wire.3dshapes/SolderWire-0.75sqmm_1x01_D1.25mm_OD3.5mm.wrl"
@@
     (fp_circle (center 0 0) (end 1.75 0)
       (stroke (width 0.1) (type solid)) (fill none) (layer "F.Fab"))
-    (pad "1" thru_hole roundrect (at 0 0) (size 3.5 3.5) (drill 1.55) (layers "*.Cu" "*.Mask") (roundrect_rratio 0.071429)
+    (pad "1" thru_hole roundrect (at 0 0) (size 3.5 3.5) (drill 1.55) (layers "*.Cu" "*.Mask") (roundrect_rratio 0.07142914286)
       (net 1 "/3v3"))
     (model "${KICAD6_3DMODEL_DIR}/Connector_Wire.3dshapes/SolderWire-0.75sqmm_1x01_D1.25mm_OD3.5mm.wrl"
@@
     (fp_circle (center 0 0) (end 1.75 0)
       (stroke (width 0.1) (type solid)) (fill none) (layer "F.Fab"))
-    (pad "1" thru_hole roundrect (at 0 0) (size 3.5 3.5) (drill 1.55) (layers "*.Cu" "*.Mask") (roundrect_rratio 0.071429)
+    (pad "1" thru_hole roundrect (at 0 0) (size 3.5 3.5) (drill 1.55) (layers "*.Cu" "*.Mask") (roundrect_rratio 0.07142914286)
       (net 58 "/9v"))
     (model "${KICAD6_3DMODEL_DIR}/Connector_Wire.3dshapes/SolderWire-0.75sqmm_1x01_D1.25mm_OD3.5mm.wrl"
